File: corne-chocolate/pcb/corne-chocolate.kicad_sch (KiCad schematic)
At the start: 88 parts, among them J1 MJ-4PP-9, J2 OLED, J3 LED, J6 Conn_01x04, P1 i2c-pin, P2 i2c-pin, SW1 SW_PUSH, SW10 SW_PUSH, SW11 SW_PUSH, SW12 SW_PUSH, SW13 SW_PUSH, SW14 SW_PUSH, SW15 SW_PUSH, SW16 SW_PUSH, SW17 SW_PUSH, SW18 SW_PUSH, SW19 SW_PUSH, SW2 SW_PUSH, SW20 SW_PUSH, SW21 SW_PUSH, SW3 SW_PUSH, SW4 SW_PUSH, SW5 SW_PUSH, SW6 SW_PUSH, SW7 SW_PUSH, SW8 SW_PUSH, SW9 SW_PUSH, U1 ProMicro

Commit message: ProMicro USB-C
Parts:
- L22, L23, L24, L25, L26, L27: footprint kbd:SK6812MINI_underglow -> kbd:SK6812MINI_underglow_rev
Connections:
- net VDD renamed +5V
